Commit message: 添加串口通信发给下位机内容
Signed-off-by: Ding Kaiyue <D570737261@163.com>

File: src/robot_description/urdf/z1.urdf.xacro (robot description, xacro)
@@ -1,5 +1,5 @@
 <robot name="z1_description" xmlns:xacro="http://www.ros.org/wiki/xacro">
-    <xacro:property name="ModelPathHead" value="file:///home/dky/Projects/z1_ws/src/robot_description/meshes/visual/" />
-    <xacro:property name="CollisionHead" value="file:///home/dky/Projects/z1_ws/src/robot_description/meshes/collision/" />
+    <xacro:property name="ModelPathHead" value="file:///home/dky/Projects/Unitree_Z1_Control/src/robot_description/meshes/visual/" />
+    <xacro:property name="CollisionHead" value="file:///home/dky/Projects/Unitree_Z1_Control/src/robot_description/meshes/collision/" />
     <xacro:include filename="$(find robot_description)/urdf/z1_const.urdf.xacro"/>
     <link name="link00">
